File: RM1xx-Breakout.sch (EAGLE design)
At the start: 25 parts, among them IC3 MCP1703, J1 JUMPER_1X30805, J6 Lipo Battery

Commit message: removed copper on mounting holes
Parts:
- removed U$9: MOUNTINGHOLE2.5, microbuilder:MOUNTINGHOLE2.5
- added U$7: MOUNTINGHOLE2.5, microbuilder:MOUNTINGHOLE2.5
Changed lines of the file:
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@@
 <part name="SUPPLY7" library="SparkFun-Aesthetics" deviceset="VCC" device="" value="3V3"/>
 <part name="GND4" library="SparkFun-Aesthetics" deviceset="GND" device=""/>
-<part name="U$3" library="microbuilder" deviceset="MOUNTINGHOLE" device="2.5"/>
-<part name="U$6" library="microbuilder" deviceset="MOUNTINGHOLE" device="2.5"/>
 <part name="NAME" library="SparkFun-Aesthetics" deviceset="FRAME-A4L" device="" value="Value">
 <attribute name="CNAME" value="RM1xx Lora+BLE breakout board"/>
@@
 <part name="VBAT" library="SparkFun-Aesthetics" deviceset="VCC" device="" value="Vbat"/>
 <part name="VBAT1" library="SparkFun-Aesthetics" deviceset="VCC" device="" value="Vbat"/>
+<part name="U$3" library="microbuilder" deviceset="MOUNTINGHOLE" device="2.5"/>
+<part name="U$6" library="microbuilder" deviceset="MOUNTINGHOLE" device="2.5"/>
+<part name="U$7" library="microbuilder" deviceset="MOUNTINGHOLE" device="2.5"/>
 <part name="U$8" library="microbuilder" deviceset="MOUNTINGHOLE" device="2.5"/>
-<part name="U$9" library="microbuilder" deviceset="MOUNTINGHOLE" device="2.5"/>
 </parts>
 <sheets>
@@
 </instance>
 <instance part="GND4" gate="1" x="104.14" y="135.255"/>
-<instance part="U$3" gate="G$1" x="13.335" y="22.86"/>
-<instance part="U$6" gate="G$1" x="13.335" y="13.97"/>
 <instance part="NAME" gate="G$1" x="4.445" y="4.445" smashed="yes">
 <attribute name="DRAWING_NAME" x="186.055" y="15.875" size="2.54" layer="94" font="vector"/>
@@
 <attribute name="VALUE" x="201.803" y="122.301" size="1.778" layer="96"/>
 </instance>
-<instance part="U$8" gate="G$1" x="20.955" y="22.86"/>
-<instance part="U$9" gate="G$1" x="20.955" y="13.97"/>
+<instance part="U$3" gate="G$1" x="14.605" y="28.575"/>
+<instance part="U$6" gate="G$1" x="21.59" y="28.575"/>
+<instance part="U$7" gate="G$1" x="27.94" y="28.575"/>
+<instance part="U$8" gate="G$1" x="34.925" y="28.575"/>
 </instances>
 <busses>

Commit message: Version 1.1
Parts:
- added C3, C4, C5: 100nF, LowPowerLab:CAP0805-CAP
- added P1: PADNORMAL, _c2h:PADNORMAL
- R6: value 390K -> 470K
- R7: value 820K -> 1M
Connections:
- net 3V3: now also C3.1, C4.2
- net CTS: now also J2.2; no longer J2.6
- net GND: now also C3.2, C4.1, C5.1
- net NARUN: now also J2.6
- net RTS: now also P1.1; no longer J2.2
- net SIO04: now also C5.2
- net VIN: now also IC3.VI; no longer IC3.VO
- net VREG: now also IC3.VO; no longer IC3.VI
Other:
- note added: "3V3"
- note added: "CTS"
- note added: "DTR"
- note added: "GND"
- note added: "RTS"
- note added: "RXD"
- note added: "TXD"
Changed lines of the file:
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@@
 <?xml version="1.0" encoding="utf-8"?>
 <!DOCTYPE eagle SYSTEM "eagle.dtd">
-<eagle version="7.6.0">
+<eagle version="7.7.0">
 <drawing>
 <settings>
@@
 <part name="NAME" library="SparkFun-Aesthetics" deviceset="FRAME-A4L" device="" value="Value">
 <attribute name="CNAME" value="RM1xx Lora+BLE breakout board"/>
-<attribute name="CREVISION" value="1.0a"/>
+<attribute name="CREVISION" value="1.1"/>
 <attribute name="DESIGNER" value="Charles-Henri Hallard"/>
 </part>
-<part name="R6" library="_c2h" deviceset="RESISTOR" device="0805-RES" value="390K"/>
-<part name="R7" library="_c2h" deviceset="RESISTOR" device="0805-RES" value="820K"/>
+<part name="R6" library="_c2h" deviceset="RESISTOR" device="0805-RES" value="470K"/>
+<part name="R7" library="_c2h" deviceset="RESISTOR" device="0805-RES" value="1M"/>
 <part name="GND5" library="SparkFun-Aesthetics" deviceset="GND" device=""/>
 <part name="VBAT" library="SparkFun-Aesthetics" deviceset="VCC" device="" value="Vbat"/>
@@
 <part name="U$7" library="microbuilder" deviceset="MOUNTINGHOLE" device="2.5"/>
 <part name="U$8" library="microbuilder" deviceset="MOUNTINGHOLE" device="2.5"/>
+<part name="C3" library="LowPowerLab" deviceset="CAP" device="0805-CAP" value="100nF"/>
+<part name="C4" library="LowPowerLab" deviceset="CAP" device="0805-CAP" value="100nF"/>
+<part name="GND6" library="SparkFun-Aesthetics" deviceset="GND" device=""/>
+<part name="GND7" library="SparkFun-Aesthetics" deviceset="GND" device=""/>
+<part name="C5" library="LowPowerLab" deviceset="CAP" device="0805-CAP" value="100nF"/>
+<part name="P1" library="_c2h" deviceset="PAD" device="NORMAL"/>
 </parts>
 <sheets>
 <sheet>
 <plain>
+<text x="67.945" y="127" size="1.778" layer="94">DTR</text>
+<text x="67.945" y="124.46" size="1.778" layer="94">RXD</text>
+<text x="67.945" y="121.92" size="1.778" layer="94">TXD</text>
+<text x="67.945" y="119.38" size="1.778" layer="94">3V3</text>
+<text x="67.945" y="116.84" size="1.778" layer="94">RTS</text>
+<text x="67.945" y="114.3" size="1.778" layer="94">GND</text>
+<text x="67.945" y="107.95" size="1.778" layer="94">CTS</text>
 </plain>
 <instances>
@@
 <attribute name="VALUE" x="117.729" y="128.016" size="1.778" layer="96"/>
 </instance>
-<instance part="IC3" gate="G$1" x="152.4" y="119.38" rot="MR0"/>
+<instance part="IC3" gate="G$1" x="152.4" y="119.38"/>
 <instance part="C2" gate="G$1" x="166.37" y="107.315" smashed="yes">
 <attribute name="NAME" x="162.814" y="110.236" size="1.778" layer="95"/>
@@
 <instance part="U$7" gate="G$1" x="27.94" y="28.575"/>
 <instance part="U$8" gate="G$1" x="34.925" y="28.575"/>
+<instance part="C3" gate="G$1" x="154.94" y="83.82" smashed="yes" rot="R90">
+<attribute name="NAME" x="155.321" y="81.534" size="1.778" layer="95" rot="R180"/>
+<attribute name="VALUE" x="156.591" y="87.884" size="1.778" layer="96" rot="R180"/>
+</instance>
+<instance part="C4" gate="G$1" x="129.54" y="83.82" smashed="yes" rot="R90">
+<attribute name="NAME" x="129.286" y="81.534" size="1.778" layer="95" rot="R180"/>
+<attribute name="VALUE" x="131.826" y="87.884" size="1.778" layer="96" rot="R180"/>
+</instance>
+<instance part="GND6" gate="1" x="120.65" y="83.82" rot="R270"/>
+<instance part="GND7" gate="1" x="161.29" y="83.82" rot="R90"/>
+<instance part="C5" gate="G$1" x="197.485" y="101.6" smashed="yes" rot="R180">
+<attribute name="NAME" x="198.501" y="104.521" size="1.778" layer="95" rot="R270"/>
+<attribute name="VALUE" x="193.421" y="103.251" size="1.778" layer="96" rot="R270"/>
+</instance>
+<instance part="P1" gate="G$1" x="76.2" y="108.585"/>
 </instances>
 <busses>
@@
 <pinref part="R7" gate="G$1" pin="1"/>
 <pinref part="GND5" gate="1" pin="GND"/>
-<wire x1="204.47" y1="95.25" x2="204.47" y2="93.98" width="0.1524" layer="91"/>
+<wire x1="204.47" y1="95.25" x2="204.47" y2="94.615" width="0.1524" layer="91"/>
+<pinref part="C5" gate="G$1" pin="1"/>
+<wire x1="204.47" y1="94.615" x2="204.47" y2="93.98" width="0.1524" layer="91"/>
+<wire x1="204.47" y1="94.615" x2="197.485" y2="94.615" width="0.1524" layer="91"/>
+<wire x1="197.485" y1="94.615" x2="197.485" y2="96.52" width="0.1524" layer="91"/>
+<junction x="204.47" y="94.615"/>
+</segment>
+<segment>
+<pinref part="C4" gate="G$1" pin="1"/>
+<pinref part="GND6" gate="1" pin="GND"/>
+<wire x1="123.19" y1="83.82" x2="124.46" y2="83.82" width="0.1524" layer="91"/>
+</segment>
+<segment>
+<pinref part="C3" gate="G$1" pin="2"/>
+<pinref part="GND7" gate="1" pin="GND"/>
+<wire x1="158.75" y1="83.82" x2="157.48" y2="83.82" width="0.1524" layer="91"/>
 </segment>
 </net>
@@
 </segment>
 <segment>
-<wire x1="83.82" y1="127" x2="94.107" y2="127" width="0.1524" layer="91"/>
-<label x="86.36" y="127" size="1.778" layer="95"/>
-<pinref part="J2" gate="G$1" pin="6"/>
-</segment>
-<segment>
 <pinref part="R2" gate="G$1" pin="1"/>
 <wire x1="241.3" y1="92.71" x2="241.3" y2="85.09" width="0.1524" layer="91"/>
@@
 <label x="88.9" y="62.23" size="1.778" layer="95"/>
 </segment>
+<segment>
+<wire x1="83.82" y1="116.84" x2="93.98" y2="116.84" width="0.1524" layer="91"/>
+<label x="86.36" y="116.84" size="1.778" layer="95"/>
+<pinref part="J2" gate="G$1" pin="2"/>
+</segment>
 </net>
 <net name="RTS" class="0">
@@
 <wire x1="120.65" y1="59.69" x2="110.49" y2="59.69" width="0.1524" layer="91"/>
 <label x="110.49" y="59.69" size="1.778" layer="95"/>
-</segment>
-<segment>
-<wire x1="83.82" y1="116.84" x2="93.98" y2="116.84" width="0.1524" layer="91"/>
-<label x="86.36" y="116.84" size="1.778" layer="95"/>
-<pinref part="J2" gate="G$1" pin="2"/>
 </segment>
 <segment>
@@
 <junction x="87.63" y="59.69"/>
 <label x="88.9" y="59.69" size="1.778" layer="95"/>
+</segment>
+<segment>
+<pinref part="P1" gate="G$1" pin="1"/>
+<wire x1="76.2" y1="108.585" x2="93.98" y2="108.585" width="0.1524" layer="91"/>
+<label x="86.36" y="108.585" size="1.778" layer="95"/>
 </segment>
 </net>
@@
 <wire x1="166.37" y1="119.38" x2="166.37" y2="112.395" width="0.1524" layer="91"/>
 <junction x="166.37" y="119.38"/>
-<pinref part="IC3" gate="G$1" pin="VI"/>
-<wire x1="162.56" y1="119.38" x2="166.37" y2="119.38" width="0.1524" layer="91"/>
 <wire x1="166.37" y1="119.38" x2="177.8" y2="119.38" width="0.1524" layer="91"/>
 <label x="167.005" y="119.38" size="1.778" layer="95"/>
+<pinref part="IC3" gate="G$1" pin="VO"/>
+<wire x1="162.56" y1="119.38" x2="166.37" y2="119.38" width="0.1524" layer="91"/>
 </segment>
 </net>
@@
 <wire x1="148.59" y1="83.82" x2="148.59" y2="74.93" width="0.1524" layer="91"/>
 <junction x="140.97" y="83.82"/>
+<pinref part="C4" gate="G$1" pin="2"/>
+<wire x1="133.35" y1="83.82" x2="132.08" y2="83.82" width="0.1524" layer="91"/>
+<pinref part="C3" gate="G$1" pin="1"/>
+<wire x1="148.59" y1="83.82" x2="149.86" y2="83.82" width="0.1524" layer="91"/>
+<junction x="133.35" y="83.82"/>
+<junction x="148.59" y="83.82"/>
 </segment>
 <segment>
@@
 <wire x1="204.47" y1="107.95" x2="204.47" y2="106.68" width="0.1524" layer="91"/>
 <wire x1="204.47" y1="106.68" x2="204.47" y2="105.41" width="0.1524" layer="91"/>
-<wire x1="204.47" y1="106.68" x2="195.58" y2="106.68" width="0.1524" layer="91"/>
-<label x="195.58" y="107.315" size="1.778" layer="95"/>
+<wire x1="204.47" y1="106.68" x2="197.485" y2="106.68" width="0.1524" layer="91"/>
+<label x="191.135" y="107.315" size="1.778" layer="95"/>
 <junction x="204.47" y="106.68"/>
+<pinref part="C5" gate="G$1" pin="2"/>
+<wire x1="197.485" y1="106.68" x2="191.135" y2="106.68" width="0.1524" layer="91"/>
+<wire x1="197.485" y1="104.14" x2="197.485" y2="106.68" width="0.1524" layer="91"/>
+<junction x="197.485" y="106.68"/>
 </segment>
 </net>
@@
 <label x="88.9" y="64.77" size="1.778" layer="95"/>
 </segment>
+<segment>
+<wire x1="83.82" y1="127" x2="94.107" y2="127" width="0.1524" layer="91"/>
+<label x="86.36" y="127" size="1.778" layer="95"/>
+<pinref part="J2" gate="G$1" pin="6"/>
+</segment>
 </net>
 <net name="VIN" class="0">
 <segment>
-<pinref part="IC3" gate="G$1" pin="VO"/>
 <pinref part="SUPPLY3" gate="1" pin="VCC"/>
 <pinref part="C1" gate="G$1" pin="1"/>
 <wire x1="119.38" y1="119.38" x2="119.38" y2="125.095" width="0.1524" layer="91"/>
-<wire x1="142.24" y1="119.38" x2="137.795" y2="119.38" width="0.1524" layer="91"/>
 <wire x1="137.795" y1="119.38" x2="119.38" y2="119.38" width="0.1524" layer="91"/>
 <wire x1="119.38" y1="114.3" x2="119.38" y2="119.38" width="0.1524" layer="91"/>
@@
 <wire x1="133.35" y1="146.685" x2="137.795" y2="146.685" width="0.1524" layer="91"/>
 <wire x1="137.795" y1="146.685" x2="137.795" y2="119.38" width="0.1524" layer="91"/>
+<label x="121.92" y="119.38" size="1.778" layer="95"/>
+<pinref part="IC3" gate="G$1" pin="VI"/>
+<wire x1="142.24" y1="119.38" x2="137.795" y2="119.38" width="0.1524" layer="91"/>
 <junction x="137.795" y="119.38"/>
-<label x="121.92" y="119.38" size="1.778" layer="95"/>
-</segment>
-</net>
+</segment>
+</net>
